File: hifi_audio.kicad_sch (KiCad schematic)
At the start: 0 parts

Commit message: update
Other:
- added sheet fonte_alimentacao (fonte_alimentacao.kicad_sch)
Changed lines of the file:
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@@
 		(rev "v1.0.0")
+	)
+	(sheet
+		(at 45.72 40.64)
+		(size 12.7 8.89)
+		(exclude_from_sim no)
+		(in_bom yes)
+		(on_board yes)
+		(dnp no)
+		(fields_autoplaced yes)
+		(stroke
+			(width 0.1524)
+			(type solid)
+		)
+		(fill
+			(color 0 0 0 0)
+		)
+		(property "Sheetname" "fonte_alimentacao"
+			(at 45.72 39.9284 0)
+			(show_name no)
+			(do_not_autoplace no)
+			(effects
+				(font
+					(size 1.27 1.27)
+				)
+				(justify left bottom)
+			)
+		)
+		(property "Sheetfile" "fonte_alimentacao.kicad_sch"
+			(at 45.72 50.1146 0)
+			(show_name no)
+			(do_not_autoplace no)
+			(effects
+				(font
+					(size 1.27 1.27)
+				)
+				(justify left top)
+			)
+		)
+		(instances
+			(project "hifi_audio"
+				(path "/cacffc98-2318-42a9-a4e2-e2aa2b951373"
+					(page "2")
+				)
+			)
+		)
 	)
 	(sheet_instances

Commit message: Definicao subbass e filtro passa baixo
Other:
- added sheet Bancada_Simulacao (Bancada_Simulacao.kicad_sch)
- added sheet subbass (subbass.kicad_sch)
Changed lines of the file:
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@@
 	)
 	(sheet
-		(at 45.72 40.64)
-		(size 12.7 8.89)
+		(at 13.97 15.24)
+		(size 12.7 6.35)
+		(exclude_from_sim no)
+		(in_bom yes)
+		(on_board yes)
+		(dnp no)
+		(fields_autoplaced yes)
+		(stroke
+			(width 0.1524)
+			(type solid)
+		)
+		(fill
+			(color 0 0 0 0)
+		)
+		(property "Sheetname" "Bancada_Simulacao"
+			(at 13.97 14.5284 0)
+			(show_name no)
+			(do_not_autoplace no)
+			(effects
+				(font
+					(size 1.27 1.27)
+				)
+				(justify left bottom)
+			)
+		)
+		(property "Sheetfile" "Bancada_Simulacao.kicad_sch"
+			(at 13.97 22.1746 0)
+			(show_name no)
+			(do_not_autoplace no)
+			(effects
+				(font
+					(size 1.27 1.27)
+				)
+				(justify left top)
+			)
+		)
+		(instances
+			(project "hifi_audio"
+				(path "/cacffc98-2318-42a9-a4e2-e2aa2b951373"
+					(page "3")
+				)
+			)
+		)
+	)
+	(sheet
+		(at 13.97 27.94)
+		(size 12.7 6.35)
 		(exclude_from_sim no)
 		(in_bom yes)
@@
 		)
 		(property "Sheetname" "fonte_alimentacao"
-			(at 45.72 39.9284 0)
+			(at 13.97 27.2284 0)
 			(show_name no)
 			(do_not_autoplace no)
@@
 		)
 		(property "Sheetfile" "fonte_alimentacao.kicad_sch"
-			(at 45.72 50.1146 0)
+			(at 13.97 34.8746 0)
 			(show_name no)
 			(do_not_autoplace no)
@@
 				)
 			)
+		)
+	)
+	(sheet
+		(at 13.97 40.64)
+		(size 12.7 6.35)
+		(exclude_from_sim no)
+		(in_bom yes)
+		(on_board yes)
+		(dnp no)
+		(fields_autoplaced yes)
+		(stroke
+			(width 0.1524)
+			(type solid)
+		)
+		(fill
+			(color 0 0 0 0)
+		)
+		(property "Sheetname" "subbass"
+			(at 13.97 39.9284 0)
+			(show_name no)
+			(do_not_autoplace no)
+			(effects
+				(font
+					(size 1.27 1.27)
+				)
+				(justify left bottom)
+			)
+		)
+		(property "Sheetfile" "subbass.kicad_sch"
+			(at 13.97 47.5746 0)
+			(show_name no)
+			(do_not_autoplace no)
+			(effects
+				(font
+					(size 1.27 1.27)
+				)
+				(justify left top)
+			)
+		)
+		(instances
+			(project "hifi_audio"
+				(path "/cacffc98-2318-42a9-a4e2-e2aa2b951373"
+					(page "4")
+				)
+			)
