File: subbass.kicad_sch (KiCad schematic)
At the start: 16 parts, among them U1 OPA1656ID

Commit message: Refactor SubBass project: Update track widths, add new connector symbols, and document modular architecture
- Reduced minimum track width and clearance in hifi_audio.kicad_pro for improved routing.
- Added new connector symbols for AUDIO_IN and AUDIO_OUT in subsbass.kicad_sch.
- Updated footprints for various components in subsbass.kicad_sch to ensure compatibility.
- Introduced modular architecture documentation in arquitetura_modular.md outlining the design and electrical interfaces.
- Created build_subbass_module_board.py script to automate PCB placement from schematic netlist.
Parts:
- added J2: AUDIO_IN, Connector_JST:JST_XH_B2B-XH-A_1x02_P2.50mm_Vertical, symbol Connector_Generic:Conn_01x02
- added J3: AUDIO_OUT, Connector_JST:JST_XH_B2B-XH-A_1x02_P2.50mm_Vertical, symbol Connector_Generic:Conn_01x02
- C1, C2, C3, C4: footprint (none) -> Capacitor_SMD:C_0805_2012Metric
- C5, C6: footprint (none) -> Capacitor_SMD:C_1206_3216Metric
- R1, R2, R3, R4: footprint (none) -> Resistor_SMD:R_0805_2012Metric
- R6: value 11,3kΩ -> 11.3k; footprint (none) -> Resistor_SMD:R_0805_2012Metric
- R7: value 22,6kΩ -> 22.6k; footprint (none) -> Resistor_SMD:R_0805_2012Metric
Connections:
- net GND: now also J2.2 (Pin_2), J3.2 (Pin_2)
- net VIN_SUB: now also J2.1 (Pin_1)
- net VOUT_SUB_MUTE: now also J3.1 (Pin_1)
Other:
- note added: "J2 AUDIO_IN (1=sinal, 2=GND); J3 AUDIO_OUT para estágio OPA1622 externo."
Changed lines of the file:
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@@
 			)
 		)
-		(property "Footprint" ""
+		(property "Footprint" "Capacitor_SMD:C_1206_3216Metric"
 			(at 167.64 95.5548 0)
 			(hide yes)
@@
 			)
 		)
-		(property "Footprint" ""
+		(property "Footprint" "Capacitor_SMD:C_0805_2012Metric"
 			(at 68.2752 111.76 0)
 			(hide yes)
@@
 			)
 		)
-		(property "Footprint" ""
+		(property "Footprint" "Resistor_SMD:R_0805_2012Metric"
 			(at 69.85 97.028 90)
 			(hide yes)
@@
 			)
 		)
-		(property "Value" "22,6kΩ"
+		(property "Value" "22.6k"
 			(at 176.53 76.2 90)
 			(show_name no)
@@
 			)
 		)
-		(property "Footprint" ""
+		(property "Footprint" "Resistor_SMD:R_0805_2012Metric"
 			(at 176.53 81.788 90)
 			(hide yes)
@@
 			)
 		)
-		(property "Footprint" ""
+		(property "Footprint" "Capacitor_SMD:C_0805_2012Metric"
 			(at 83.82 81.5848 0)
 			(hide yes)
@@
 			)
 		)
-		(property "Footprint" ""
+		(property "Footprint" "Resistor_SMD:R_0805_2012Metric"
 			(at 158.242 171.45 90)
 			(hide yes)
@@
 			)
 		)
-		(property "Value" "11,3kΩ"
+		(property "Value" "11.3k"
 			(at 179.832 106.172 90)
 			(show_name no)
@@
 			)
 		)
-		(property "Footprint" ""
+		(property "Footprint" "Resistor_SMD:R_0805_2012Metric"
 			(at 182.88 99.822 90)
 			(hide yes)
@@
 			)
 		)
-		(property "Footprint" ""
+		(property "Footprint" "Resistor_SMD:R_0805_2012Metric"
 			(at 52.07 97.028 90)
 			(hide yes)
@@
 			)
 		)
-		(property "Footprint" ""
+		(property "Footprint" "Resistor_SMD:R_0805_2012Metric"
 			(at 130.302 171.45 90)
 			(hide yes)
@@
 			)
 		)
-		(property "Footprint" ""
+		(property "Footprint" "Capacitor_SMD:C_0805_2012Metric"
 			(at 164.7952 140.97 0)
 			(hide yes)
@@
 			)
 		)
-		(property "Footprint" ""
+		(property "Footprint" "Capacitor_SMD:C_0805_2012Metric"
 			(at 127.9652 140.97 0)
 			(hide yes)
@@
 			)
 		)
-		(property "Footprint" ""
+		(property "Footprint" "Capacitor_SMD:C_1206_3216Metric"
 			(at 180.34 95.5548 0)
 			(hide yes)
@@
 (symbol (lib_id "Audio_HiFi:TESTPOINT") (at 269.24 78.74 0) (unit 1) (exclude_from_sim yes) (in_bom no) (on_board yes) (property "Reference" "TP1" (at 269.24 74.92999999999999 0) (effects (font (size 1 1)))) (property "Value" "TestPoint" (at 269.24 78.74 0) (hide yes) (effects (font (size 1 1)))) (property "Footprint" "TestPoint:TestPoint_Pad_D1.5mm" (at 269.24 78.74 0) (hide yes) (effects (font (size 1 1)))) (pin "1") (instances (project "hifi_audio" (path "/cacffc98-2318-42a9-a4e2-e2aa2b951373/ad6bf775-41d3-4b77-b1e8-7e04674efb8f" (reference "TP1") (unit 1)))))
 (symbol (lib_id "Audio_HiFi:TESTPOINT") (at 269.24 90.17 0) (unit 1) (exclude_from_sim yes) (in_bom no) (on_board yes) (property "Reference" "TP2" (at 269.24 86.36 0) (effects (font (size 1 1)))) (property "Value" "TestPoint" (at 269.24 90.17 0) (hide yes) (effects (font (size 1 1)))) (property "Footprint" "TestPoint:TestPoint_Pad_D1.5mm" (at 269.24 90.17 0) (hide yes) (effects (font (size 1 1)))) (pin "1") (instances (project "hifi_audio" (path "/cacffc98-2318-42a9-a4e2-e2aa2b951373/ad6bf775-41d3-4b77-b1e8-7e04674efb8f" (reference "TP2") (unit 1)))))
+(symbol (lib_id "Connector_Generic:Conn_01x02") (at 360.68 149.86 0) (unit 1) (body_style 1) (exclude_from_sim no) (in_bom yes) (on_board yes) (in_pos_files yes) (dnp no) (fields_autoplaced yes)
+(property "Reference" "J2" (at 365.76 147.32000000000002 0) (effects (font (size 1.27 1.27)) (justify left)))
+(property "Value" "AUDIO_IN" (at 365.76 149.86 0) (effects (font (size 1.27 1.27)) (justify left)))
+(property "Footprint" "Connector_JST:JST_XH_B2B-XH-A_1x02_P2.50mm_Vertical" (at 360.68 149.86 0) (hide yes) (effects (font (size 1.27 1.27))))
+(property "Datasheet" "https://www.jst-mfg.com/product/index.php?series=287" (at 360.68 149.86 0) (hide yes) (effects (font (size 1.27 1.27))))
+(pin "1") (pin "2")
+(instances (project "hifi_audio" (path "/cacffc98-2318-42a9-a4e2-e2aa2b951373/ad6bf775-41d3-4b77-b1e8-7e04674efb8f" (reference "J2") (unit 1)))))
+(symbol (lib_id "Connector_Generic:Conn_01x02") (at 360.68 170.18 0) (unit 1) (body_style 1) (exclude_from_sim no) (in_bom yes) (on_board yes) (in_pos_files yes) (dnp no) (fields_autoplaced yes)
+(property "Reference" "J3" (at 365.76 167.64000000000001 0) (effects (font (size 1.27 1.27)) (justify left)))
+(property "Value" "AUDIO_OUT" (at 365.76 170.18 0) (effects (font (size 1.27 1.27)) (justify left)))
+(property "Footprint" "Connector_JST:JST_XH_B2B-XH-A_1x02_P2.50mm_Vertical" (at 360.68 170.18 0) (hide yes) (effects (font (size 1.27 1.27))))
+(property "Datasheet" "https://www.jst-mfg.com/product/index.php?series=287" (at 360.68 170.18 0) (hide yes) (effects (font (size 1.27 1.27))))
+(pin "1") (pin "2")
+(instances (project "hifi_audio" (path "/cacffc98-2318-42a9-a4e2-e2aa2b951373/ad6bf775-41d3-4b77-b1e8-7e04674efb8f" (reference "J3") (unit 1)))))
+(wire (pts (xy 355.6 149.86) (xy 342.9 149.86)) (stroke (width 0) (type default)))
+(label "VIN_SUB" (at 342.9 149.86 180) (effects (font (size 1 1)) (justify right bottom)))
+(wire (pts (xy 355.6 170.18) (xy 342.9 170.18)) (stroke (width 0) (type default)))
+(label "VOUT_SUB_MUTE" (at 342.9 170.18 180) (effects (font (size 1 1)) (justify right bottom)))
+(text "J2 AUDIO_IN (1=sinal, 2=GND); J3 AUDIO_OUT para estágio OPA1622 externo." (at 294.64 180.34 0) (effects (font (size 1 1)) (justify left top)))
+(symbol
+		(lib_id "power:GND")
+		(at 355.6 152.4 0)
+		(unit 1)
+		(body_style 1)
+		(exclude_from_sim no)
+		(in_bom yes)
+		(on_board yes)
+		(in_pos_files yes)
+		(dnp no)
+		(fields_autoplaced yes)
+		(property "Reference" "#PWR050"
+			(at 355.6 152.4 0)
+			(hide yes)
+			(show_name no)
+			(do_not_autoplace no)
+			(effects
+				(font
+					(size 1.27 1.27)
+				)
+			)
+		)
+		(property "Value" "GND"
+			(at 355.6 152.4 0)
+			(show_name no)
+			(do_not_autoplace no)
+			(effects
+				(font
+					(size 1.27 1.27)
+				)
+			)
+		)
+		(property "Footprint" ""
+			(at 355.6 152.4 0)
+			(hide yes)
+			(show_name no)
+			(do_not_autoplace no)
+			(effects
+				(font
+					(size 1.27 1.27)
+				)
+			)
+		)
+		(property "Datasheet" ""
+			(at 355.6 152.4 0)
+			(hide yes)
+			(show_name no)
+			(do_not_autoplace no)
+			(effects
+				(font
+					(size 1.27 1.27)
+				)
+			)
+		)
+		(property "Description" "Power symbol creates a global label with name \"GND\" , ground"
+			(at 355.6 152.4 0)
+			(hide yes)
+			(show_name no)
+			(do_not_autoplace no)
+			(effects
+				(font
+					(size 1.27 1.27)
+				)
+			)
+		)
+		(pin "1"
+		)
+		(instances
+			(project "hifi_audio"
+				(path "/cacffc98-2318-42a9-a4e2-e2aa2b951373/ad6bf775-41d3-4b77-b1e8-7e04674efb8f"
+					(reference "#PWR050")
+					(unit 1)
+				)
+			)
+		)
+	)(symbol
+		(lib_id "power:GND")
+		(at 355.6 172.72 0)
+		(unit 1)
+		(body_style 1)
+		(exclude_from_sim no)
+		(in_bom yes)
+		(on_board yes)
+		(in_pos_files yes)
+		(dnp no)
+		(fields_autoplaced yes)
+		(property "Reference" "#PWR051"
+			(at 355.6 172.72 0)
+			(hide yes)
+			(show_name no)
+			(do_not_autoplace no)
+			(effects
+				(font
+					(size 1.27 1.27)
+				)
+			)
+		)
+		(property "Value" "GND"
+			(at 355.6 172.72 0)
+			(show_name no)
+			(do_not_autoplace no)
+			(effects
+				(font
+					(size 1.27 1.27)
+				)
+			)
+		)
+		(property "Footprint" ""
+			(at 355.6 172.72 0)
+			(hide yes)
+			(show_name no)
+			(do_not_autoplace no)
+			(effects
+				(font
+					(size 1.27 1.27)
+				)
+			)
+		)
+		(property "Datasheet" ""
+			(at 355.6 172.72 0)
+			(hide yes)
+			(show_name no)
+			(do_not_autoplace no)
+			(effects
+				(font
+					(size 1.27 1.27)
+				)
+			)
+		)
+		(property "Description" "Power symbol creates a global label with name \"GND\" , ground"
+			(at 355.6 172.72 0)
+			(hide yes)
+			(show_name no)
+			(do_not_autoplace no)
+			(effects
+				(font
+					(size 1.27 1.27)
+				)
+			)
+		)
+		(pin "1"
+		)
+		(instances
+			(project "hifi_audio"
+				(path "/cacffc98-2318-42a9-a4e2-e2aa2b951373/ad6bf775-41d3-4b77-b1e8-7e04674efb8f"
+					(reference "#PWR051")
+					(unit 1)
+				)
+			)
+		)
+	)
 )

Commit message: Ajustes e limpeza
Other:
- note removed: "Filtros concluídos em SPICE. Mute físico: protótipo e ensaios de bancada pendentes."
- note removed: "J2 AUDIO_IN (1=sinal, 2=GND); J3 AUDIO_OUT para estágio OPA1622 externo."
- note removed: "Mute físico em folha filha: LTC2909 + ADG5412F. Modelos locais de estudo."
- note removed: "U1A: passa-baixas ~40 Hz"
- note removed: "U1B: passa-altas ~10 Hz"
- note removed: "U4: supervisão +UV/-UV; U5: chave protegida. Ver detalhes na folha Mute_SubBass."
- moved on the sheet: C3, C4, C5, C6, J2, J3, R3, R4, R6, R7, TP1, TP2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
